File: eagle/hrem.sch (EAGLE design)
At the start: 7 parts, among them U1 TINY85-20-DIP

Commit message: PCB improvements
Parts:
- removed C1: 22uF, SparkFun-Capacitors:CAPKIT
- removed G1: CR2032H, battery:CR2032H
- added BAT1: (no value), SparkFun-Electromechanical:BATTERYAAA
- added C2: 10uF, SparkFun-Capacitors:10UF-16V-10%(TANT)
- added C3: 100uF, SparkFun-Capacitors:10UF-16V-10%(TANT)
- added C4: 22uF, SparkFun-Capacitors:10UF-16V-10%(TANT)
- added L1: 47uH, SparkFun-Passives:INDUCTORCR54-47UH
- added R2: 300K, SparkFun-Resistors:RESISTOR1206
- added R3: 100K, SparkFun-Resistors:RESISTOR1206
- added R4: 100, SparkFun-Resistors:RESISTOR1206
- added U$1: LM2621SMD, SparkFun-PowerIC:LM2621SMD
- LED1: device led:LED3MM -> led:LEDSML1206
- R1: device SparkFun-Resistors:RESISTORPTH-1/4W -> SparkFun-Resistors:RESISTOR1206
- U1: value TINY85-20-DIP -> Tiny85-20-SMT; device SparkFun-DigitalIC:ATTINY45TINY85-20-DIP -> SparkFun-DigitalIC:ATTINY45TINY85-20-SMT
Connections:
- new net N$10: C2.-, R4.2, U$1.SW
- new net N$12: R2.2, R3.1, U$1.FB
- new net N$15: BAT1.+, C4.+, L1.1, R4.1
- new net N$9: C2.+, L1.2, U$1.FREQ
- net GND: now also BAT1.-, C3.-, C4.-, R3.2, U$1.PGND, U$1.SGND; no longer C1.2, G1.-
- net N$3: now also U1.PB4(ADC2); no longer U1.PB3(ADC3)
- net N$5: now also U1.PB3(ADC3); no longer U1.PB4(ADC2)
- net VCC: now also C3.+, R2.1, U$1.BOOT, U$1.EN, U$1.VDD; no longer C1.1, G1.+

Commit message: SMD version
Parts:
- removed C2: 10uF, SparkFun-Capacitors:10UF-16V-10%(TANT)
- added C1: 4.7pF, rcl:C-EUC1206
- added D1: CGRM4001-G, diode:CGRM4001-G
- added R5: 100K, SparkFun-Resistors:RESISTOR1206
- C3: device SparkFun-Capacitors:10UF-16V-10%(TANT) -> rcl:C-EUC1206
- C4: device SparkFun-Capacitors:10UF-16V-10%(TANT) -> rcl:CPOL-EUE2.5-5
- L1: value 47uH -> 4.7uH
- LED1: device led:LEDSML1206 -> led:LED3MM
- R1: value 100 -> 200
- R4: value 100 -> 150K
Connections:
- new net N$11: C1.2, R4.1, U$1.FREQ
- new net N$2: R5.1, U1.PB5(NRES)
- net GND: now also C3.2; no longer C3.-
- net N$10: now also L1.2; no longer C2.-, U$1.SW
- net N$15: no longer L1.1, R4.1
- net N$9: now also C1.1, D1.A, L1.1, U$1.SW; no longer C2.+, L1.2, U$1.FREQ
- net VCC: now also C3.1, D1.C, R5.2; no longer C3.+, U1.PB5(NRES)
Other:
- moved on the sheet: L1, R4
