File: hardware/hrem/hrem.sch (KiCad schematic (older format))
At the start: 17 parts

Commit message: hardware changes
Parts:
- removed U?: HT7733, symbol hrem:HT7733
- added U1: HT7733A, symbol hrem:HT7733A
- added U3: 74AHC1G125, symbol 74xGxx:74AHC1G125
- added U4: 74LVC1G125, symbol 74xGxx:74AHC1G125
- C2: renamed from C?; value 100uF -> 22uF
- gave numbers to parts that had none: 15
Connections:
- net labels added: PE
- wire segments 58 -> 80
Other:
- note added: "Programming Header"
- note added: "Vcc = 3.3V"
- moved on the sheet: BZ1, D2, J2, L1, Q1, R1, R2, R3, SW2

Commit message: Some changes to schematics
Parts:
- added C3: 100nF, symbol Device:C
Connections:
- net labels removed: PE
- wire segments 80 -> 84
Other:
- moved on the sheet: SW2
Changed lines of the file:
@@
 Sheet 1 1
 Title "HRem"
-Date "2019-10-10"
-Rev ""
+Date "2019-10-25"
+Rev "4"
 Comp "Denis Bazhenov"
 Comment1 ""
@@
 L power:VCC #PWR0106
 U 1 1 5DA7C60F
-P 7000 1400
-F 0 "#PWR0106" H 7000 1250 50  0001 C CNN
-F 1 "VCC" H 7017 1573 50  0000 C CNN
-F 2 "" H 7000 1400 50  0001 C CNN
-F 3 "" H 7000 1400 50  0001 C CNN
-	1    7000 1400
+P 7000 1250
+F 0 "#PWR0106" H 7000 1100 50  0001 C CNN
+F 1 "VCC" H 7017 1423 50  0000 C CNN
+F 2 "" H 7000 1250 50  0001 C CNN
+F 3 "" H 7000 1250 50  0001 C CNN
+	1    7000 1250
 	1    0    0    -1
 $EndComp
@@
 L Switch:SW_Push SW2
 U 1 1 5DA2030D
-P 8950 1050
-F 0 "SW2" H 8950 1250 50  0000 C CNN
-F 1 "SW_Push" H 8950 1244 50  0001 C CNN
-F 2 "" H 8950 1250 50  0001 C CNN
-F 3 "~" H 8950 1250 50  0001 C CNN
-	1    8950 1050
+P 8950 950
+F 0 "SW2" H 8950 1150 50  0000 C CNN
+F 1 "SW_Push" H 8950 1144 50  0001 C CNN
+F 2 "" H 8950 1150 50  0001 C CNN
+F 3 "~" H 8950 1150 50  0001 C CNN
+	1    8950 950
 	1    0    0    -1
 $EndComp
@@
 	7600 1850 7900 1850
 Wire Wire Line
-	7900 1850 7900 1050
-Wire Wire Line
-	7900 1050 8750 1050
-Wire Wire Line
-	9150 1050 9250 1050
-Wire Wire Line
-	9250 1050 9250 1400
+	7900 1850 7900 950
+Wire Wire Line
+	7900 950  8750 950
+Wire Wire Line
+	9150 950  9250 950
+Wire Wire Line
+	9250 950  9250 1400
 $Comp
 L Switch:SW_DIP_x01 SW1
@@
 	8500 2000 8500 1950
 Wire Wire Line
-	8400 1850 8400 1800
-Wire Wire Line
-	8400 1800 8500 1800
-Wire Wire Line
-	8400 1200 8400 1150
-Wire Wire Line
-	8400 1150 8500 1150
-Text Label 8400 1150 0    50   ~ 0
-PE
-Text Label 8400 1800 0    50   ~ 0
-PE
+	8400 1850 8400 1700
+Wire Wire Line
+	8400 1700 8450 1700
+Wire Wire Line
+	8400 1200 8400 1050
+Wire Wire Line
+	8400 1050 8450 1050
 Wire Wire Line
 	8900 2050 8900 2400
@@
 Text Notes 7950 4850 0    50   ~ 10
 Programming Header
+$Comp
+L power:GND #PWR02
+U 1 1 5DB4FF74
+P 8450 1050
+F 0 "#PWR02" H 8450 800 50  0001 C CNN
+F 1 "GND" V 8450 850 50  0000 C CNN
+F 2 "" H 8450 1050 50  0001 C CNN
+F 3 "" H 8450 1050 50  0001 C CNN
+	1    8450 1050
+	0    -1   -1   0
+$EndComp
+$Comp
+L power:GND #PWR03
+U 1 1 5DB56A1F
+P 8450 1700
+F 0 "#PWR03" H 8450 1450 50  0001 C CNN
+F 1 "GND" V 8450 1500 50  0000 C CNN
+F 2 "" H 8450 1700 50  0001 C CNN
+F 3 "" H 8450 1700 50  0001 C CNN
+	1    8450 1700
+	0    -1   -1   0
+$EndComp
+$Comp
+L Device:C C3
+U 1 1 5DB6C80A
+P 6700 1400
+F 0 "C3" V 6448 1400 50  0000 C CNN
+F 1 "100nF" V 6539 1400 50  0000 C CNN
+F 2 "" H 6738 1250 50  0001 C CNN
+F 3 "~" H 6700 1400 50  0001 C CNN
+	1    6700 1400
+	0    1    1    0
+$EndComp
+Wire Wire Line
+	6850 1400 7000 1400
+Connection ~ 7000 1400
+Wire Wire Line
+	7000 1400 7000 1250
+$Comp
+L power:GND #PWR01
+U 1 1 5DB724EA
+P 6250 1450
+F 0 "#PWR01" H 6250 1200 50  0001 C CNN
+F 1 "GND" H 6255 1277 50  0000 C CNN
+F 2 "" H 6250 1450 50  0001 C CNN
+F 3 "" H 6250 1450 50  0001 C CNN
+	1    6250 1450
+	1    0    0    -1
+$EndComp
+Wire Wire Line
+	6250 1450 6250 1400
+Wire Wire Line
+	6250 1400 6550 1400
 $EndSCHEMATC

Commit message: New rev
Parts:
- added R4: 100R, symbol Device:R
Connections:
- wire segments 84 -> 86
Other:
- moved on the sheet: SW2
Changed lines of the file:
@@
 Sheet 1 1
 Title "HRem"
-Date "2019-10-25"
-Rev "4"
+Date "2019-11-24"
+Rev "5"
 Comp "Denis Bazhenov"
 Comment1 ""
@@
 U 1 1 5D9F2256
 P 7000 2150
-F 0 "U2" H 6600 2700 50  0000 R CNN
-F 1 "ATtiny85" H 7500 2700 50  0000 R CNN
+F 0 "U2" H 6470 2196 50  0000 R CNN
+F 1 "ATtiny85" H 6470 2105 50  0000 R CNN
 F 2 "Package_SO:SOIJ-8_5.3x5.3mm_P1.27mm" H 7000 2150 50  0001 C CIN
 F 3 "http://ww1.microchip.com/downloads/en/DeviceDoc/atmel-2586-avr-8-bit-microcontroller-attiny25-attiny45-attiny85_datasheet.pdf" H 7000 2150 50  0001 C CNN
@@
 U 1 1 5D9F4947
 P 1850 1900
-F 0 "BT1" H 1700 2000 50  0000 R CNN
-F 1 "1xAAA" H 1700 1900 50  0000 R CNN
+F 0 "BT1" H 1968 1996 50  0000 L CNN
+F 1 "1xAAA" H 1968 1905 50  0000 L CNN
 F 2 "" V 1850 1960 50  0001 C CNN
 F 3 "~" V 1850 1960 50  0001 C CNN
@@
 U 1 1 5DA03F1D
 P 9150 1400
-F 0 "D2" H 9150 1200 50  0000 C CNN
-F 1 "LED" H 9150 1300 50  0000 C CNN
+F 0 "D2" H 9150 1195 50  0000 C CNN
+F 1 "LED" H 9150 1286 50  0000 C CNN
 F 2 "" V 9150 1400 50  0001 C CNN
 F 3 "~" V 9150 1400 50  0001 C CNN
@@
 U 1 1 5DA9218E
 P 8850 1400
-F 0 "R3" V 8950 1300 50  0000 L CNN
-F 1 "68R" V 8750 1300 50  0000 L CNN
+F 0 "R3" V 8950 1400 50  0000 L CNN
+F 1 "68R" V 8750 1350 50  0000 L CNN
 F 2 "" V 8780 1400 50  0001 C CNN
 F 3 "~" H 8850 1400 50  0001 C CNN
@@
 $EndComp
 Wire Wire Line
-	7600 1950 8050 1950
+	7600 1950 8000 1950
 $Comp
 L power:GND #PWR0107
@@
 L Switch:SW_Push SW2
 U 1 1 5DA2030D
-P 8950 950
-F 0 "SW2" H 8950 1150 50  0000 C CNN
-F 1 "SW_Push" H 8950 1144 50  0001 C CNN
-F 2 "" H 8950 1150 50  0001 C CNN
-F 3 "~" H 8950 1150 50  0001 C CNN
-	1    8950 950
-	1    0    0    -1
-$EndComp
-Wire Wire Line
-	7600 1850 7900 1850
-Wire Wire Line
-	7900 1850 7900 950
-Wire Wire Line
-	7900 950  8750 950
-Wire Wire Line
-	9150 950  9250 950
-Wire Wire Line
-	9250 950  9250 1400
+P 7900 1550
+F 0 "SW2" H 7900 1743 50  0000 C CNN
+F 1 "SW_Push" H 7900 1744 50  0001 C CNN
+F 2 "" H 7900 1750 50  0001 C CNN
+F 3 "~" H 7900 1750 50  0001 C CNN
+	1    7900 1550
+	0    -1   -1   0
+$EndComp
 $Comp
 L Switch:SW_DIP_x01 SW1
 U 1 1 5DA31AB0
 P 2200 1600
-F 0 "SW1" H 2200 1800 50  0000 C CNN
+F 0 "SW1" H 2200 1775 50  0000 C CNN
 F 1 "POWER_SWITCH" H 2200 1776 50  0001 C CNN
 F 2 "" H 2200 1600 50  0001 C CNN
@@
 	9000 1400 9050 1400
 $Comp
-L 74xGxx:74AHC1G125 U4
-U 1 1 5DB16C1F
-P 8400 2050
-F 0 "U4" H 8250 2250 50  0000 C CNN
-F 1 "74LVC1G125" H 8850 2100 50  0000 C CNN
-F 2 "" H 8400 2050 50  0001 C CNN
-F 3 "http://www.ti.com/lit/sg/scyt129e/scyt129e.pdf" H 8400 2050 50  0001 C CNN
-	1    8400 2050
-	1    0    0    -1
-$EndComp
-$Comp
 L power:VCC #PWR0113
 U 1 1 5DB25976
@@
 	8500 2000 8500 1950
 Wire Wire Line
-	8400 1850 8400 1700
-Wire Wire Line
-	8400 1700 8450 1700
-Wire Wire Line
-	8400 1200 8400 1050
-Wire Wire Line
-	8400 1050 8450 1050
+	8400 1850 8400 1750
+Wire Wire Line
+	8400 1750 8450 1750
 Wire Wire Line
 	8900 2050 8900 2400
@@
 Wire Wire Line
 	8450 2350 8450 2500
-Connection ~ 9250 1400
-Wire Wire Line
-	8050 1400 8100 1400
-Wire Wire Line
-	8050 1400 8050 1950
+Wire Wire Line
+	8000 1400 8100 1400
+Wire Wire Line
+	8000 1400 8000 1950
 Wire Wire Line
 	9250 1400 9250 1500
@@
 U 1 1 5D9F300D
 P 8450 3300
-F 0 "BZ1" V 8750 3200 50  0000 L CNN
-F 1 "Buzzer" V 8650 3200 50  0000 L CNN
+F 0 "BZ1" V 8647 3282 50  0000 C CNN
+F 1 "Buzzer" V 8738 3282 50  0000 C CNN
 F 2 "" V 8425 3400 50  0001 C CNN
 F 3 "~" V 8425 3400 50  0001 C CNN
@@
 Wire Wire Line
 	8800 2300 8800 2400
-Wire Wire Line
-	7600 2050 8100 2050
 Wire Wire Line
 	8650 2050 8900 2050
@@
 U 1 1 5DC3B268
 P 3900 2050
-F 0 "U1" V 3550 1850 50  0000 L CNN
-F 1 "HT7733A" V 3550 2000 50  0000 L CNN
+F 0 "U1" V 3577 2100 50  0000 C CNN
+F 1 "HT7733A" V 3486 2100 50  0000 C CNN
 F 2 "" H 3900 2000 50  0001 C CNN
 F 3 "https://datasheet.lcsc.com/szlcsc/Holtek-Semicon-HT7733A_C131130.pdf" H 3900 2000 50  0001 C CNN
@@
 L power:VCC #PWR0116
 U 1 1 5DA7DA17
-P 8650 3100
-F 0 "#PWR0116" H 8650 2950 50  0001 C CNN
-F 1 "VCC" H 8667 3273 50  0000 C CNN
-F 2 "" H 8650 3100 50  0001 C CNN
-F 3 "" H 8650 3100 50  0001 C CNN
-	1    8650 3100
+P 8950 3100
+F 0 "#PWR0116" H 8950 2950 50  0001 C CNN
+F 1 "VCC" H 8967 3273 50  0000 C CNN
+F 2 "" H 8950 3100 50  0001 C CNN
+F 3 "" H 8950 3100 50  0001 C CNN
+	1    8950 3100
 	1    0    0    -1
 $EndComp
 Wire Wire Line
 	8550 3200 8550 3150
-Wire Wire Line
-	8550 3150 8650 3150
-Wire Wire Line
-	8650 3150 8650 3100
 Wire Wire Line
 	8050 2850 8050 2700
@@
 U 1 1 5D9F33C3
 P 8050 3050
-F 0 "Q1" V 8300 2950 50  0000 L CNN
-F 1 "BC547" V 8400 2950 50  0000 L CNN
+F 0 "Q1" V 8285 3050 50  0000 C CNN
+F 1 "BC547" V 8376 3050 50  0000 C CNN
 F 2 "Package_TO_SOT_THT:TO-92_Inline" H 8250 2975 50  0001 L CIN
 F 3 "http://www.fairchildsemi.com/ds/BC/BC547.pdf" H 8050 3050 50  0001 L CNN
@@
 L power:GND #PWR02
 U 1 1 5DB4FF74
-P 8450 1050
-F 0 "#PWR02" H 8450 800 50  0001 C CNN
-F 1 "GND" V 8450 850 50  0000 C CNN
-F 2 "" H 8450 1050 50  0001 C CNN
-F 3 "" H 8450 1050 50  0001 C CNN
-	1    8450 1050
+P 8450 1100
+F 0 "#PWR02" H 8450 850 50  0001 C CNN
+F 1 "GND" V 8450 900 50  0000 C CNN
+F 2 "" H 8450 1100 50  0001 C CNN
+F 3 "" H 8450 1100 50  0001 C CNN
+	1    8450 1100
 	0    -1   -1   0
 $EndComp
@@
 L power:GND #PWR03
 U 1 1 5DB56A1F
-P 8450 1700
-F 0 "#PWR03" H 8450 1450 50  0001 C CNN
-F 1 "GND" V 8450 1500 50  0000 C CNN
-F 2 "" H 8450 1700 50  0001 C CNN
-F 3 "" H 8450 1700 50  0001 C CNN
-	1    8450 1700
+P 8450 1750
+F 0 "#PWR03" H 8450 1500 50  0001 C CNN
+F 1 "GND" V 8450 1550 50  0000 C CNN
+F 2 "" H 8450 1750 50  0001 C CNN
+F 3 "" H 8450 1750 50  0001 C CNN
+	1    8450 1750
 	0    -1   -1   0
 $EndComp
@@
 Wire Wire Line
 	6250 1400 6550 1400
+$Comp
+L Device:R R4
+U 1 1 5DB85F94
+P 8750 3150
+F 0 "R4" V 8850 3150 50  0000 L CNN
+F 1 "100R" V 8650 3050 50  0000 L CNN
+F 2 "" V 8680 3150 50  0001 C CNN
+F 3 "~" H 8750 3150 50  0001 C CNN
+	1    8750 3150
+	0    -1   -1   0
+$EndComp
+Wire Wire Line
+	8550 3150 8600 3150
+Wire Wire Line
+	8900 3150 8950 3150
+Wire Wire Line
+	8950 3150 8950 3100
+Wire Wire Line
+	7900 2050 7600 2050
+Wire Wire Line
+	8100 2050 8100 1850
+Wire Wire Line
+	8100 1850 7600 1850
+$Comp
+L 74xGxx:74AHC1G125 U4
+U 1 1 5DB16C1F
+P 8400 2050
+F 0 "U4" H 8250 2250 50  0000 C CNN
+F 1 "74LVC1G125" H 8850 2100 50  0000 C CNN
+F 2 "" H 8400 2050 50  0001 C CNN
+F 3 "http://www.ti.com/lit/sg/scyt129e/scyt129e.pdf" H 8400 2050 50  0001 C CNN
+	1    8400 2050
+	1    0    0    -1
+$EndComp
+Wire Wire Line
+	8400 1100 8450 1100
+Wire Wire Line
+	8400 1200 8400 1100
+Wire Wire Line
+	7900 2050 7900 1750
+$Comp
+L power:GND #PWR?
+U 1 1 5DDF8B2E
+P 7500 1200
+F 0 "#PWR?" H 7500 950 50  0001 C CNN
+F 1 "GND" H 7505 1027 50  0000 C CNN
+F 2 "" H 7500 1200 50  0001 C CNN
+F 3 "" H 7500 1200 50  0001 C CNN
+	1    7500 1200
+	1    0    0    -1
+$EndComp
+Wire Wire Line
+	7900 1350 7900 1150
+Wire Wire Line
+	7900 1150 7500 1150
+Wire Wire Line
+	7500 1150 7500 1200
 $EndSCHEMATC

Commit message: Migration to new KiCad version
Parts:
- removed J1: ICSP, symbol Connector_Generic:Conn_02x03_Counter_Clockwise
- removed SW1: POWER_SWITCH, symbol Switch:SW_DIP_x01
- removed SW2: SW_Push, symbol Switch:SW_Push
- removed U3: 74AHC1G125, symbol 74xGxx:74AHC1G125
- removed U4: 74LVC1G125, symbol 74xGxx:74AHC1G125
- added J1: ICSP, Connector_PinSocket_2.54mm:PinSocket_2x05_P2.54mm_Vertical, symbol Connector_Generic:Conn_02x05_Odd_Even
- added SW1: SW_Push_Dual, hrem:button, symbol Switch:SW_Push_Dual
- BT1: footprint (none) -> Battery:BatteryHolder_Keystone_2466_1xAAA
- BZ1: footprint (none) -> hrem:buzzer
- C1, C2, C3: footprint (none) -> Capacitor_THT:CP_Radial_D5.0mm_P2.50mm
- D2: footprint (none) -> LED_THT:LED_D5.0mm
- J2: footprint (none) -> Connector_JST:JST_EH_B3B-EH-A_1x03_P2.50mm_Vertical
- L1: footprint (none) -> Inductor_THT:L_Axial_L5.3mm_D2.2mm_P7.62mm_Horizontal_Vishay_IM-1
- Q1: footprint Package_TO_SOT_THT:TO-92_Inline -> Package_TO_SOT_THT:TO-92_Inline_Wide
- R1, R2, R3, R4: footprint (none) -> Resistor_THT:R_Axial_DIN0207_L6.3mm_D2.5mm_P7.62mm_Horizontal
- U1: footprint (none) -> hrem:HT7733
- U2: footprint Package_SO:SOIJ-8_5.3x5.3mm_P1.27mm -> Package_DIP:DIP-8_W7.62mm_Socket; symbol MCU_Microchip_ATtiny:ATtiny85-20SU -> hrem-rescue:ATtiny85-20SU-MCU_Microchip_ATtiny
Connections:
- wire segments 86 -> 81
- no-connect marks 0 -> 1

Commit message: Update ICSP footprint information
Parts:
- J1: footprint Connector_PinSocket_2.54mm:PinSocket_2x05_P2.54mm_Vertical -> Connector_IDC:IDC-Header_2x05_P2.54mm_Vertical
Changed lines of the file:
@@
 F 0 "J1" H 8400 5867 50  0000 C CNN
 F 1 "ICSP" H 8400 5776 50  0000 C CNN
-F 2 "Connector_PinSocket_2.54mm:PinSocket_2x05_P2.54mm_Vertical" H 8350 5450 50  0001 C CNN
+F 2 "Connector_IDC:IDC-Header_2x05_P2.54mm_Vertical" H 8350 5450 50  0001 C CNN
 F 3 "~" H 8350 5450 50  0001 C CNN
 	1    8350 5450
