File: hardware/hrem/hrem.sch (KiCad schematic (older format))
At the start: 29 parts, among them J1 AVR-ISP, J2 Hall_Conn, Q1 MMBT4401-7-F, SW1 SW_Push_Dual, U1 HT7733A, U2 ATtiny85, U3 74LVC1G125, U4 74LVC1G125

Commit message: PCB ref names positioning and vendor part names
Parts:
- C1: Part TAJB476K010RNJ -> C22036; Vendor (none) -> TAJB476K010RNJ
- C2: Part TAJB226K010RNJ -> C7198; Vendor (none) -> TAJB226K010RNJ
- D1: Vendor (none) -> SS14-E3/61T
- J2: Vendor (none) -> X8821WRS-03-9TSN
- L1: Vendor (none) -> LQH43CN101K03L
- Q1: Vendor (none) -> MMBT4401-7-F
- R1: Vendor (none) -> RTT051002FTP
- R2: Vendor (none) -> ERJ6ENF6800V
- R3, R4: Vendor (none) -> ERJ6ENF1000V
- R5, R6: Vendor (none) -> CR-05JA7----0R
- SW1: Vendor (none) -> DTSM-65N-V-T/R
- U3, U4: Vendor (none) -> SN74LVC1G125DBVR
Changed lines of the file:
@@
 F 3 "https://datasheet.lcsc.com/szlcsc/1906141836_XKB-Enterprise-X8821WRS-03-9TSN_C397433.pdf" H 8750 4100 50  0001 C CNN
 F 4 "C397433" H 8750 4100 50  0001 C CNN "Part"
+F 5 "X8821WRS-03-9TSN" H 8750 4100 50  0001 C CNN "Vendor"
 	1    8750 4100
 	0    1    -1   0
@@
 F 2 "Capacitor_Tantalum_SMD:CP_EIA-3528-15_AVX-H_Pad1.50x2.35mm_HandSolder" H 1838 1550 50  0001 C CNN
 F 3 "https://datasheet.lcsc.com/szlcsc/AVX-TAJB476K010RNJ_C22036.pdf" H 1800 1700 50  0001 C CNN
-F 4 "TAJB476K010RNJ" H 1800 1700 50  0001 C CNN "Part"
+F 4 "C22036" H 1800 1700 50  0001 C CNN "Part"
+F 5 "TAJB476K010RNJ" H 1800 1700 50  0001 C CNN "Vendor"
 	1    1800 1700
 	1    0    0    -1
@@
 F 2 "Capacitor_Tantalum_SMD:CP_EIA-3528-15_AVX-H_Pad1.50x2.35mm_HandSolder" H 3738 1650 50  0001 C CNN
 F 3 "https://datasheet.lcsc.com/szlcsc/AVX-TAJB226K010RNJ_C7198.pdf" H 3700 1800 50  0001 C CNN
-F 4 "TAJB226K010RNJ" H 3700 1800 50  0001 C CNN "Part"
+F 4 "C7198" H 3700 1800 50  0001 C CNN "Part"
+F 5 "TAJB226K010RNJ" H 3700 1800 50  0001 C CNN "Vendor"
 	1    3700 1800
 	1    0    0    -1
@@
 F 3 "https://datasheet.lcsc.com/szlcsc/Vishay-Intertech-SS14-E3-61T_C47460.pdf" H 2950 1450 50  0001 C CNN
 F 4 "C47460" H 2950 1450 50  0001 C CNN "Part"
+F 5 "SS14-E3/61T" H 2950 1450 50  0001 C CNN "Vendor"
 	1    2950 1450
 	-1   0    0    1
@@
 F 3 "~" H 7600 4050 50  0001 C CNN
 F 4 "C410034" H 7600 4050 50  0001 C CNN "Part"
+F 5 "ERJ6ENF6800V" H 7600 4050 50  0001 C CNN "Vendor"
 	1    7600 4050
 	-1   0    0    1
@@
 F 3 "~" H 7300 4050 50  0001 C CNN
 F 4 "C103904" H 7300 4050 50  0001 C CNN "Part"
+F 5 "RTT051002FTP" H 7300 4050 50  0001 C CNN "Vendor"
 	1    7300 4050
 	-1   0    0    1
@@
 F 3 "https://datasheet.lcsc.com/szlcsc/Murata-Electronics-LQH43CN101K03L_C113087.pdf" H 2150 1450 50  0001 C CNN
 F 4 "C113087" H 2150 1450 50  0001 C CNN "Part"
+F 5 "LQH43CN101K03L" H 2150 1450 50  0001 C CNN "Vendor"
 	1    2150 1450
 	1    0    0    -1
@@
 F 3 "https://datasheet.lcsc.com/szlcsc/Diodes-Incorporated-MMBT4401-7-F_C151826.pdf" H 7600 4550 50  0001 L CNN
 F 4 "C151826" V 7600 4550 50  0001 C CNN "Part"
+F 5 "MMBT4401-7-F" H 7600 4550 50  0001 C CNN "Vendor"
 	1    7600 4550
 	0    1    1    0
@@
 F 3 "~" H 8300 4650 50  0001 C CNN
 F 4 "C193990" H 8300 4650 50  0001 C CNN "Part"
+F 5 "ERJ6ENF1000V" H 8300 4650 50  0001 C CNN "Vendor"
 	1    8300 4650
 	0    -1   -1   0
@@
 F 3 "https://datasheet.lcsc.com/szlcsc/Diptronics-DTSM-65N-V-T-R_C224982.pdf" H 7150 2900 50  0001 C CNN
 F 4 "C224982" H 7150 2700 50  0001 C CNN "Part"
+F 5 "DTSM-65N-V-T/R" H 7150 2700 50  0001 C CNN "Vendor"
 	1    7150 2700
 	1    0    0    -1
@@
 F 3 "https://datasheet.lcsc.com/szlcsc/Texas-Instruments-TI-SN74LVC1G125DBVR_C23654.pdf" H 8400 3350 50  0001 C CNN
 F 4 "C23654" H 8400 3350 50  0001 C CNN "Part"
+F 5 "SN74LVC1G125DBVR" H 8400 3350 50  0001 C CNN "Vendor"
 	1    8400 3350
 	1    0    0    -1
@@
 F 3 "https://datasheet.lcsc.com/szlcsc/2001071207_Viking-Tech-CR-05JA7-0R_C465486.pdf" H 8200 3550 50  0001 C CNN
 F 4 "C465486" H 8200 3550 50  0001 C CNN "Part"
+F 5 "CR-05JA7----0R" H 8200 3550 50  0001 C CNN "Vendor"
 	1    8200 3550
 	0    -1   -1   0
@@
 F 3 "https://datasheet.lcsc.com/szlcsc/2001071207_Viking-Tech-CR-05JA7-0R_C465486.pdf" H 8000 1500 50  0001 C CNN
 F 4 "C465486" H 8000 1500 50  0001 C CNN "Part"
+F 5 "CR-05JA7----0R" H 8000 1500 50  0001 C CNN "Vendor"
 	1    8000 1500
 	0    -1   -1   0
@@
 F 3 "https://datasheet.lcsc.com/szlcsc/Texas-Instruments-TI-SN74LVC1G125DBVR_C23654.pdf" H 7900 2200 50  0001 C CNN
 F 4 "C23654" H 7900 2200 50  0001 C CNN "Part"
+F 5 "SN74LVC1G125DBVR" H 7900 2200 50  0001 C CNN "Vendor"
 	1    7900 2200
 	1    0    0    -1
@@
 F 3 "~" H 8600 2200 50  0001 C CNN
 F 4 "C193990" H 8600 2200 50  0001 C CNN "Part"
+F 5 "ERJ6ENF1000V" H 8600 2200 50  0001 C CNN "Vendor"
 	1    8600 2200
 	0    -1   -1   0

Commit message: Fixed layout issue
Q1 has invalid schematics symbol. Base and collector was swaped.
Parts:
- removed Q1: MMBT4401-7-F, Package_TO_SOT_SMD:SOT-23_Handsoldering, symbol Transistor_BJT:BC547
- added Q1: MMBT4401-7-F, Package_TO_SOT_SMD:SOT-23_Handsoldering, symbol Device:Q_NPN_BCE
Connections:
- net GND: now also Q1.3 (E)
- net at BZ1.2 (+): now also Q1.2 (C)
- net at R2.1, TP3.1: now also Q1.1 (B)
Changed lines of the file:
@@
 Wire Wire Line
 	7600 4350 7600 4300
-$Comp
-L Transistor_BJT:BC547 Q1
-U 1 1 5D9F33C3
-P 7600 4550
-F 0 "Q1" V 7850 4550 50  0000 C CNN
-F 1 "MMBT4401-7-F" V 7500 4950 50  0001 C CNN
-F 2 "Package_TO_SOT_SMD:SOT-23_Handsoldering" H 7800 4475 50  0001 L CIN
-F 3 "https://datasheet.lcsc.com/szlcsc/Diodes-Incorporated-MMBT4401-7-F_C151826.pdf" H 7600 4550 50  0001 L CNN
-F 4 "C151826" V 7600 4550 50  0001 C CNN "Part"
-F 5 "MMBT4401-7-F" H 7600 4550 50  0001 C CNN "Vendor"
-	1    7600 4550
-	0    1    1    0
-$EndComp
 Text Notes 1500 4950 0    50   ~ 10
 Programming Header
@@
 Wire Wire Line
 	8100 3650 7150 3650
+$Comp
+L Device:Q_NPN_BCE Q1
+U 1 1 5E99FA84
+P 7600 4550
+F 0 "Q1" V 7836 4550 50  0000 C CNN
+F 1 "MMBT4401-7-F" V 7926 4550 50  0001 C CNN
+F 2 "Package_TO_SOT_SMD:SOT-23_Handsoldering" H 7800 4650 50  0001 C CNN
+F 3 "https://datasheet.lcsc.com/szlcsc/Diodes-Incorporated-MMBT4401-7-F_C151826.pdf~" H 7600 4550 50  0001 C CNN
+F 4 "C151826" H 7600 4550 50  0001 C CNN "Part"
+F 5 "MMBT4401-7-F" H 7600 4550 50  0001 C CNN "Vendor"
+	1    7600 4550
+	0    1    1    0
+$EndComp
 $EndSCHEMATC
