File: hardware/hrem/hrem.kicad_pcb (KiCad board)
At the start: 2 copper layers, 80 x 44.4 mm, 31 parts, among them J1 AVR-ISP, J2 Hall_Conn, Q1 MMBT4401-7-F, SW1 SW_Push_Dual, U1 HT7733A, U2 ATtiny85, U3 74LVC1G125, U4 74LVC1G125

Commit message: PCB tracks cleanup
Parts:
- moved TP2 8.58 mm to (69.8, 64.9)
Routing:
- net VCC: track 48.9 -> 41.1 mm
- net Net-(J2-Pad2): track 49.8 -> 45.3 mm
- net /MISO: track 48.9 -> 46.2 mm
- net /SCK: track 52.4 -> 50.7 mm
- net Net-(R2-Pad2): track 13.7 -> 13.0 mm
Changed lines of the file:
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@@
     (thickness 1.6)
     (drawings 14)
-    (tracks 181)
+    (tracks 175)
     (zones 0)
     (modules 31)
@@
   )
   (module TestPoint:TestPoint_Pad_D2.0mm (layer F.Cu)
-    (at 62.103 68.58)
+    (at 69.85 64.897)
     (descr "SMD pad as test Point, diameter 2.0mm")
     (tags "test point SMD pad")
@@
   (via (at 113.3425 60.706) (size 0.5) (drill 0.3) (layers F.Cu B.Cu) (net 4))
   (segment (start 113.3425 63.1495) (end 113.3425 59.436) (width 0.5) (layer B.Cu) (net 4))
-  (segment (start 63.517213 68.58) (end 69.85 68.58) (width 0.5) (layer F.Cu) (net 4))
-  (segment (start 62.103 68.58) (end 63.517213 68.58) (width 0.5) (layer F.Cu) (net 4))
   (segment (start 69.85 74.422) (end 69.85 68.58) (width 0.5) (layer F.Cu) (net 4))
   (segment (start 69.85 68.58) (end 69.85 59.309) (width 0.5) (layer F.Cu) (net 4))
@@
   (segment (start 77.47 76.962) (end 78.658601 78.150601) (width 0.25) (layer B.Cu) (net 10))
   (segment (start 80.599399 78.150601) (end 83.25751 75.49249) (width 0.25) (layer B.Cu) (net 10))
-  (segment (start 77.978 62.357) (end 77.978 62.357) (width 0.25) (layer F.Cu) (net 10))
-  (via (at 77.978 62.357) (size 0.5) (drill 0.3) (layers F.Cu B.Cu) (net 10))
-  (segment (start 76.835 62.357) (end 77.978 62.357) (width 0.25) (layer F.Cu) (net 10))
-  (segment (start 76.118601 63.073399) (end 76.835 62.357) (width 0.25) (layer F.Cu) (net 10))
-  (segment (start 77.47 76.962) (end 76.118601 75.610601) (width 0.25) (layer F.Cu) (net 10))
-  (segment (start 76.118601 75.610601) (end 76.118601 63.073399) (width 0.25) (layer F.Cu) (net 10))
   (segment (start 83.25751 75.49249) (end 101.01949 75.49249) (width 0.25) (layer B.Cu) (net 10))
   (segment (start 101.473 75.946) (end 101.473 78.0415) (width 0.25) (layer B.Cu) (net 10))
   (segment (start 101.01949 75.49249) (end 101.473 75.946) (width 0.25) (layer B.Cu) (net 10))
+  (via (at 78.74 62.611) (size 0.5) (drill 0.3) (layers F.Cu B.Cu) (net 10))
+  (segment (start 78.74 75.692) (end 78.74 62.611) (width 0.25) (layer F.Cu) (net 10))
+  (segment (start 77.47 76.962) (end 78.74 75.692) (width 0.25) (layer F.Cu) (net 10))
   (segment (start 112.3925 67.3735) (end 112.3925 65.8495) (width 0.25) (layer B.Cu) (net 11) (status 20))
   (segment (start 112.2045 66.8835) (end 112.4585 66.6295) (width 0.25) (layer F.Cu) (net 11) (status 30))
-  (segment (start 101.4975 79.3115) (end 102.8065 79.3115) (width 0.25) (layer F.Cu) (net 11))
   (segment (start 80.137 76.962) (end 80.01 76.962) (width 0.25) (layer B.Cu) (net 11))
-  (segment (start 103.505 78.613) (end 103.505 74.803) (width 0.25) (layer F.Cu) (net 11))
-  (segment (start 102.8065 79.3115) (end 103.505 78.613) (width 0.25) (layer F.Cu) (net 11))
   (segment (start 80.01 76.962) (end 82.169 74.803) (width 0.25) (layer B.Cu) (net 11))
   (segment (start 82.169 74.803) (end 103.505 74.803) (width 0.25) (layer B.Cu) (net 11))
@@
   (segment (start 112.3925 68.1965) (end 112.3925 68.1965) (width 0.25) (layer B.Cu) (net 11))
   (via (at 112.3925 68.1965) (size 0.5) (drill 0.3) (layers F.Cu B.Cu) (net 11))
-  (segment (start 112.3925 72.2655) (end 112.3925 68.1965) (width 0.25) (layer F.Cu) (net 11))
-  (segment (start 103.505 74.803) (end 109.855 74.803) (width 0.25) (layer F.Cu) (net 11))
-  (segment (start 109.855 74.803) (end 112.3925 72.2655) (width 0.25) (layer F.Cu) (net 11))
   (segment (start 112.3925 66.6955) (end 112.4585 66.6295) (width 0.25) (layer F.Cu) (net 11))
   (segment (start 112.3925 68.1965) (end 112.3925 66.6955) (width 0.25) (layer F.Cu) (net 11))
-  (segment (start 126.1745 69.723) (end 129.6035 69.723) (width 0.25) (layer F.Cu) (net 12) (status 10))
-  (segment (start 129.6035 69.723) (end 130.2385 70.358) (width 0.25) (layer F.Cu) (net 12))
-  (segment (start 130.2385 70.358) (end 130.2385 77.343) (width 0.25) (layer F.Cu) (net 12))
-  (segment (start 130.2385 77.343) (end 129.7305 77.851) (width 0.25) (layer F.Cu) (net 12))
-  (segment (start 129.7305 77.851) (end 125.712 77.851) (width 0.25) (layer F.Cu) (net 12) (status 20))
+  (segment (start 110.1115 68.1965) (end 103.505 74.803) (width 0.25) (layer F.Cu) (net 11))
+  (segment (start 112.3925 68.1965) (end 110.1115 68.1965) (width 0.25) (layer F.Cu) (net 11))
+  (segment (start 102.2975 79.3115) (end 101.4975 79.3115) (width 0.25) (layer F.Cu) (net 11))
+  (segment (start 103.505 74.803) (end 103.505 78.104) (width 0.25) (layer F.Cu) (net 11))
+  (segment (start 103.505 78.104) (end 102.2975 79.3115) (width 0.25) (layer F.Cu) (net 11))
   (segment (start 95.0975 78.0415) (end 96.99251 79.93651) (width 0.25) (layer F.Cu) (net 12))
   (segment (start 94.2975 78.0415) (end 95.0975 78.0415) (width 0.25) (layer F.Cu) (net 12))
@@
   (segment (start 103.702501 80.588501) (end 103.05051 79.93651) (width 0.25) (layer F.Cu) (net 12))
   (segment (start 120.164001 80.588501) (end 103.702501 80.588501) (width 0.25) (layer F.Cu) (net 12))
+  (segment (start 127.174499 70.722999) (end 126.1745 69.723) (width 0.25) (layer F.Cu) (net 12))
+  (segment (start 128.287001 71.835501) (end 127.174499 70.722999) (width 0.25) (layer F.Cu) (net 12))
+  (segment (start 128.287001 77.775999) (end 128.287001 71.835501) (width 0.25) (layer F.Cu) (net 12))
+  (segment (start 125.712 77.851) (end 128.212 77.851) (width 0.25) (layer F.Cu) (net 12))
+  (segment (start 128.212 77.851) (end 128.287001 77.775999) (width 0.25) (layer F.Cu) (net 12))
   (segment (start 94.759213 66.802) (end 96.139 66.802) (width 0.25) (layer F.Cu) (net 13))
   (segment (start 93.345 66.802) (end 94.759213 66.802) (width 0.25) (layer F.Cu) (net 13))
-  (segment (start 93.17249 78.98649) (end 93.17249 70.02251) (width 0.25) (layer F.Cu) (net 14))
+  (segment (start 95.439 68.852) (end 96.139 68.852) (width 0.25) (layer F.Cu) (net 14))
+  (segment (start 93.17249 71.11851) (end 95.439 68.852) (width 0.25) (layer F.Cu) (net 14))
+  (segment (start 93.17249 78.98649) (end 93.17249 71.11851) (width 0.25) (layer F.Cu) (net 14))
   (segment (start 94.2975 79.3115) (end 93.4975 79.3115) (width 0.25) (layer F.Cu) (net 14))
   (segment (start 93.4975 79.3115) (end 93.17249 78.98649) (width 0.25) (layer F.Cu) (net 14))
-  (segment (start 94.343 68.852) (end 96.139 68.852) (width 0.25) (layer F.Cu) (net 14))
-  (segment (start 93.17249 70.02251) (end 94.343 68.852) (width 0.25) (layer F.Cu) (net 14))
   (segment (start 118.646 80.391) (end 118.6485 80.3885) (width 0.25) (layer B.Cu) (net 17) (status 30))
   (segment (start 116.0145 80.391) (end 118.646 80.391) (width 0.25) (layer B.Cu) (net 17) (status 30))
@@
   (segment (start 119.888 75.7555) (end 120.2925 75.351) (width 0.25) (layer F.Cu) (net 17))
   (segment (start 120.2925 75.351) (end 125.712 75.351) (width 0.25) (layer F.Cu) (net 17) (status 20))
+  (segment (start 123.212 75.351) (end 125.712 75.351) (width 0.25) (layer F.Cu) (net 17))
+  (segment (start 121.9835 69.723) (end 121.9835 74.1225) (width 0.25) (layer F.Cu) (net 17))
   (segment (start 121.9835 74.1225) (end 123.212 75.351) (width 0.25) (layer F.Cu) (net 17))
-  (segment (start 123.212 75.351) (end 125.712 75.351) (width 0.25) (layer F.Cu) (net 17) (status 20))
-  (segment (start 121.9835 69.723) (end 121.9835 74.1225) (width 0.25) (layer F.Cu) (net 17) (status 10))
   (via (at 110.4265 62.6745) (size 0.5) (drill 0.3) (layers F.Cu B.Cu) (net 18))
   (via (at 110.4265 63.5635) (size 0.5) (drill 0.3) (layers F.Cu B.Cu) (net 18))
